Commit message: feat: migrate selected arm driver updates

File: software/ros2/src/openeai_arm_urdf_ros2/urdf/STEP.urdf (robot description, URDF)
Before this commit: robot STEP, 7 links, 6 joints
Links:
- link link2: mass 1.5389 -> 1.3679
- link link3: mass 1.01598 -> 0.9137
- link link4: mass 0.53515 -> 0.7251
- link link5: mass 0.46797 -> 0.5538
- link link6: mass 0.83362 -> 0.3720
